File: eagle/teensy36-test-harness-4.brd (EAGLE design)
At the start: 78.2 x 50 mm, 5 parts

Commit message: Add files via upload
Parts:
- added JGND, JMIDI: (no value), SparkFun-Connectors:1X08
- moved JPWR 63.1 mm to (29.4, -4.97)
- moved JTFT 41.5 mm to (63.4, 26.4)
- moved JDIO 10.3 mm to (49.6, 28.5)
- moved JAIO 0.81 mm to (21.1, 40.6)
Connections:
- new net AREF: JMIDI.5, U$3.AREF
- net 3V3: now also JMIDI.3, U$3.3V3
- net GND: now also JGND.1, JGND.2, JGND.3, JGND.4, JGND.5, JGND.6, JGND.7, JGND.8, JMIDI.6, JMIDI.7, JMIDI.8
- net MIDI_RX: now also JMIDI.1
- net MIDI_TX: now also JMIDI.2
- net VIN: now also JMIDI.4
Routing:
- net 3V3: track 0.00 -> 56.7 mm
- net MIDI_TX: track 48.8 -> 95.3 mm, vias 0 -> 1
- net SPI0_SCLK: track 74.2 -> 32.0 mm
- net TFT_RST: track 70.6 -> 30.2 mm
- net MIDI_RX: track 41.1 -> 79.1 mm, vias 1 -> 0
- net SPI0_MOSI: track 42.7 -> 13.6 mm
- net T2: track 17.7 -> 40.6 mm
- net TFT_CS: track 37.4 -> 18.7 mm
- net T30: track 26.5 -> 12.4 mm
- net T3: track 14.1 -> 28.2 mm
- net TA20: track 52.6 -> 39.3 mm
- net AREF: track 0.00 -> 12.7 mm
- net TA19: track 47.6 -> 35.7 mm
- net T4: track 15.1 -> 26.3 mm, vias 0 -> 1
- net TA18: track 42.9 -> 32.1 mm
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Other:
- board size 78.2 x 50 mm -> 78.2 x 58.5 mm
- board text added: "Analog IO"
- board text added: "Digital I/O"
- board text added: "MIDI"
- board text added: "TFT"
